File: pcb/cert-datalogger.kicad_pcb (KiCad board)
At the start: 2 copper layers, 27.5 x 43.5 mm, 33 parts, among them IC1 ESP32-C3-MINI-1-H4, J1 Header 01x02 2.54mm, J2 Header 01x04 2.54mm, J3 Header 01x02 2.54mm, J4 Header 01x02 2.54mm, Q1 S8550, U1 LPS22HB, U3 W25X40CLSN, U4 TLV75533PDBV

Commit message: Fix ESP32 3D model
Parts:
- IC1: value ESP32-C3-MINI-1-H4 -> ESP32C3MINI1H4
